Commit message: Change the urdf file to "DFQ_right_hand.urdf" and retest it

File: anyteleop/robot/g1_description/inspire_hand_viz.urdf (robot description, URDF)
Before this commit: robot inspire_hand_left, 13 links, 12 joints
Links:
- removed link L_hand_base_link
- removed link L_index_intermediate
- removed link L_index_proximal
- removed link L_middle_intermediate
- removed link L_middle_proximal
- removed link L_pinky_intermediate
- removed link L_pinky_proximal
- removed link L_ring_intermediate
- removed link L_ring_proximal
- removed link L_thumb_distal
- removed link L_thumb_intermediate
- removed link L_thumb_proximal
- removed link L_thumb_proximal_base
- added link R_hand_base_link, mass 0.14143; collision mesh filename=meshes/R_hand_base_link.STL; visual mesh filename=meshes/R_hand_base_link.STL
- added link R_index_intermediate, mass 0.0045683; collision mesh filename=meshes/Link16_R.STL; visual mesh filename=meshes/Link16_R.STL
- added link R_index_proximal, mass 0.0042403; collision mesh filename=meshes/Link15_R.STL; visual mesh filename=meshes/Link15_R.STL
- added link R_middle_intermediate, mass 0.0050396; collision mesh filename=meshes/Link18_R.STL; visual mesh filename=meshes/Link18_R.STL
- added link R_middle_proximal, mass 0.0042403; collision mesh filename=meshes/Link17_R.STL; visual mesh filename=meshes/Link17_R.STL
- added link R_pinky_intermediate, mass 0.0035996; collision mesh filename=meshes/Link22_R.STL; visual mesh filename=meshes/Link22_R.STL
- added link R_pinky_proximal, mass 0.0042403; collision mesh filename=meshes/Link21_R.STL; visual mesh filename=meshes/Link21_R.STL
- added link R_ring_intermediate, mass 0.0045683; collision mesh filename=meshes/Link20_R.STL; visual mesh filename=meshes/Link20_R.STL
- added link R_ring_proximal, mass 0.0042403; collision mesh filename=meshes/Link19_R.STL; visual mesh filename=meshes/Link19_R.STL
- added link R_thumb_distal, mass 0.0033441; collision mesh filename=meshes/Link14_R.STL; visual mesh filename=meshes/Link14_R.STL
- added link R_thumb_intermediate, mass 0.0037847; collision mesh filename=meshes/Link13_R.STL; visual mesh filename=meshes/Link13_R.STL
- added link R_thumb_proximal, mass 0.0066075; collision mesh filename=meshes/Link12_R.STL; visual mesh filename=meshes/Link12_R.STL
- added link R_thumb_proximal_base, mass 0.0018869; collision mesh filename=meshes/Link11_R.STL; visual mesh filename=meshes/Link11_R.STL
- added link right_wrist_yaw_link
Joints:
- removed joint L_index_intermediate_joint
- removed joint L_index_proximal_joint
- removed joint L_middle_intermediate_joint
- removed joint L_middle_proximal_joint
- removed joint L_pinky_intermediate_joint
- removed joint L_pinky_proximal_joint
- removed joint L_ring_intermediate_joint
- removed joint L_ring_proximal_joint
- removed joint L_thumb_distal_joint
- removed joint L_thumb_intermediate_joint
- removed joint L_thumb_proximal_pitch_joint
- removed joint L_thumb_proximal_yaw_joint
- added joint R_base_link_joint: type fixed, parent right_wrist_yaw_link, child R_hand_base_link, origin xyz=0.0415 0 0 rpy=3.1415926535897932384626433832795 0 -1.5707963267948966192313216916398
- added joint R_index_intermediate_joint: type revolute, parent R_index_proximal, child R_index_intermediate, origin xyz=-0.0026138 0.032026 -0.001 rpy=0 0 0, axis 0 0 1, limit lower=0 upper=1.7 effort=1 velocity=0.5, mimic joint=R_index_proximal_joint multiplier=1 offset=0
- added joint R_index_proximal_joint: type revolute, parent R_hand_base_link, child R_index_proximal, origin xyz=0.00028533 -0.13653 -0.032268 rpy=-3.1067 0 0, axis 0 0 1, limit lower=0 upper=1.7 effort=1 velocity=0.5
- added joint R_middle_intermediate_joint: type revolute, parent R_middle_proximal, child R_middle_intermediate, origin xyz=-0.0024229 0.032041 -0.001 rpy=0 0 0, axis 0 0 1, limit lower=0 upper=1.7 effort=1 velocity=0.5, mimic joint=R_middle_proximal_joint multiplier=1 offset=0
- added joint R_middle_proximal_joint: type revolute, parent R_hand_base_link, child R_middle_proximal, origin xyz=0.00028533 -0.1371 -0.01295 rpy=-3.1416 0 0, axis 0 0 1, limit lower=0 upper=1.7 effort=1 velocity=0.5
- added joint R_pinky_intermediate_joint: type revolute, parent R_pinky_proximal, child R_pinky_intermediate, origin xyz=-0.0024229 0.032041 -0.001 rpy=0 0 0, axis 0 0 1, limit lower=0 upper=1.7 effort=1 velocity=0.5, mimic joint=R_pinky_proximal_joint multiplier=1 offset=0
- added joint R_pinky_proximal_joint: type revolute, parent R_hand_base_link, child R_pinky_proximal, origin xyz=0.00028533 -0.13571 0.025488 rpy=3.0369 0 0, axis 0 0 1, limit lower=0 upper=1.7 effort=1 velocity=0.5
- added joint R_ring_intermediate_joint: type revolute, parent R_ring_proximal, child R_ring_intermediate, origin xyz=-0.0024229 0.032041 -0.001 rpy=0 0 0, axis 0 0 1, limit lower=0 upper=1.7 effort=1 velocity=0.5, mimic joint=R_ring_proximal_joint multiplier=1 offset=0
- added joint R_ring_proximal_joint: type revolute, parent R_hand_base_link, child R_ring_proximal, origin xyz=0.00028533 -0.13691 0.0062872 rpy=3.0892 0 0, axis 0 0 1, limit lower=0 upper=1.7 effort=1 velocity=0.5
- added joint R_thumb_distal_joint: type revolute, parent R_thumb_intermediate, child R_thumb_distal, origin xyz=0.020248 0.010156 -0.0012 rpy=0 0 0, axis 0 0 1, limit lower=0 upper=1.2 effort=1 velocity=0.5, mimic joint=R_thumb_proximal_pitch_joint multiplier=2.4 offset=0
- added joint R_thumb_intermediate_joint: type revolute, parent R_thumb_proximal, child R_thumb_intermediate, origin xyz=0.04407 0.034553 -0.0008 rpy=0 0 0, axis 0 0 1, limit lower=0 upper=0.8 effort=1 velocity=0.5, mimic joint=R_thumb_proximal_pitch_joint multiplier=1.6 offset=0
- added joint R_thumb_proximal_pitch_joint: type revolute, parent R_thumb_proximal_base, child R_thumb_proximal, origin xyz=-0.0088099 0.010892 -0.00925 rpy=1.5708 0 2.8587, axis 0 0 1, limit lower=-0.1 upper=0.6 effort=1 velocity=0.5
- added joint R_thumb_proximal_yaw_joint: type revolute, parent R_hand_base_link, child R_thumb_proximal_base, origin xyz=-0.01696 -0.0691 -0.02045 rpy=1.5708 -1.5708 0, axis 0 0 -1, limit lower=-0.1 upper=1.3 effort=1 velocity=0.5
